File: motor_test.kicad_pcb (KiCad board)
At the start: 2 copper layers, 40 parts, among them J1 Conn_01x02_Male, J2 Conn_01x01_Male, J3 Conn_01x01_Male, J4 Conn_01x02_Male, Q1 BC817, Q10 FR024N, Q11 BC807, Q12 BC817, Q13 BC817, Q14 BC817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

Commit message: bistable
Parts:
- added Q17: BC817, Package_TO_SOT_SMD:SOT-23, F.Cu at (232.7, 51.7)
- added Q18: BC817, Package_TO_SOT_SMD:SOT-23, F.Cu at (232.7, 56.2)
- added R17: 1k, Resistor_SMD:R_1206_3216Metric, F.Cu at (217.4, 59.2)
- added R18: 1k, Resistor_SMD:R_1206_3216Metric, F.Cu at (227.6, 51.0)
- added R19: 10k, Resistor_SMD:R_1206_3216Metric, F.Cu at (223.0, 59.2)
- added R20: 10k, Resistor_SMD:R_1206_3216Metric, F.Cu at (227.6, 54.3)

Commit message: bistable
Parts:
- added D5: 1N4148, Diode_THT:D_DO-35_SOD27_P7.62mm_Horizontal, F.Cu at (247.7, 22.2)
- added D6: 1N4148, Diode_THT:D_DO-35_SOD27_P7.62mm_Horizontal, F.Cu at (247.7, 25.8)
- added J2: Conn_01x02_Male, Connector_PinHeader_2.54mm:PinHeader_1x02_P2.54mm_Vertical, F.Cu at (199.9, 18.4)
- added R21: 100k, Resistor_SMD:R_1206_3216Metric, F.Cu at (259.6, 22.1)
- added R22: 100k, Resistor_SMD:R_1206_3216Metric, F.Cu at (248.9, 29.2)
- added R23: 100k, Resistor_SMD:R_1206_3216Metric, F.Cu at (259.6, 25.4)
- moved J3 210.3 mm to (51.2, 68.8)
Connections:
- net Net-(Q17-Pad1) renamed RST
- J2 pad 1: FWD,REV -> (no net)
- Q16 pad 1: Net-(Q1-Pad1) -> Net-(Q16-Pad1)
- Q16 pad 2: Net-(Q14-Pad1) -> GNDREF
- Q16 pad 3: Net-(D1-Pad1) -> Net-(Q14-Pad1)
- Q17 pad 2: Net-(Q17-Pad2) -> GNDREF
- Q18 pad 2: Net-(Q17-Pad2) -> GNDREF
- R1 pad 1: Net-(Q1-Pad1) -> REV
- R1 pad 2: FWD,REV -> Net-(Q1-Pad1)
- R16 pad 1: GNDREF -> Net-(Q14-Pad1)
- R16 pad 2: Net-(Q14-Pad1) -> Net-(D1-Pad1)
- R17 pad 2: Net-(R17-Pad2) -> Net-(D1-Pad1)
- R18 pad 2: Net-(R17-Pad2) -> Net-(D1-Pad1)

Commit message: nightly
Parts:
- added D1: 1N4148, Diode_THT:D_DO-35_SOD27_P7.62mm_Horizontal, F.Cu at (104.9, 34.9)
- added D1: 1N4148, Diode_THT:D_DO-35_SOD27_P7.62mm_Horizontal, F.Cu at (244.9, 85.2)
- added D10: 1N4148, Diode_THT:D_DO-35_SOD27_P7.62mm_Horizontal, F.Cu at (295.1, 72.7)
- added D2: 1N4148, Diode_THT:D_DO-35_SOD27_P7.62mm_Horizontal, F.Cu at (104.9, 38.5)
- added D2: 1N4148, Diode_THT:D_DO-35_SOD27_P7.62mm_Horizontal, F.Cu at (257.0, 69.1)
- added D7: 1N4148, Diode_THT:D_DO-35_SOD27_P7.62mm_Horizontal, F.Cu at (257.0, 95.4)
- added D8: 1N4148, Diode_THT:D_DO-35_SOD27_P7.62mm_Horizontal, F.Cu at (257.0, 91.9)
- added D9: 1N4148, Diode_THT:D_DO-35_SOD27_P7.62mm_Horizontal, F.Cu at (295.1, 69.1)
- added J5: Conn_01x02_Male, Connector_PinHeader_2.54mm:PinHeader_1x02_P2.54mm_Vertical, F.Cu at (257.8, 73.2)
- added Q1: BC817, Package_TO_SOT_SMD:SOT-23, F.Cu at (96.5, 35.4)
- added Q1: BC817, Package_TO_SOT_SMD:SOT-23, F.Cu at (273.5, 77.5)
- added Q19: BC807, Package_TO_SOT_SMD:SOT-23, F.Cu at (263.3, 102.8)
- added Q2: BC817, Package_TO_SOT_SMD:SOT-23, F.Cu at (96.5, 40.0)
- added Q2: BC817, Package_TO_SOT_SMD:SOT-23, F.Cu at (268.9, 79.7)
- added Q20: FR9024N, Package_TO_SOT_SMD:TO-252-3_TabPin2, F.Cu at (249.4, 102.2)
- added Q21: BC817, Package_TO_SOT_SMD:SOT-23, F.Cu at (267.7, 103.5)
- added Q22: BC807, Package_TO_SOT_SMD:SOT-23, F.Cu at (273.3, 100.2)
- added Q23: BC817, Package_TO_SOT_SMD:SOT-23, F.Cu at (263.3, 107.3)
- added Q24: FR024N, Package_TO_SOT_SMD:TO-252-3_TabPin2, F.Cu at (249.4, 94.1)
- added Q25: BC817, Package_TO_SOT_SMD:SOT-23, F.Cu at (268.9, 98.9)
- added Q26: BC817, Package_TO_SOT_SMD:SOT-23, F.Cu at (274.0, 95.7)
- added Q27: BC807, Package_TO_SOT_SMD:SOT-23, F.Cu at (305.8, 80.7)
- added Q28: FR9024N, Package_TO_SOT_SMD:TO-252-3_TabPin2, F.Cu at (287.5, 71.4)
- added Q29: BC817, Package_TO_SOT_SMD:SOT-23, F.Cu at (311.4, 77.5)
- added Q30: BC807, Package_TO_SOT_SMD:SOT-23, F.Cu at (301.4, 84.6)
- added Q31: BC817, Package_TO_SOT_SMD:SOT-23, F.Cu at (307.0, 76.2)
- added Q32: FR024N, Package_TO_SOT_SMD:TO-252-3_TabPin2, F.Cu at (287.5, 79.4)
- added Q33: BC817, Package_TO_SOT_SMD:SOT-23, F.Cu at (312.1, 72.9)
- added Q34: BC817, Package_TO_SOT_SMD:SOT-23, F.Cu at (301.4, 80.0)
- added Q4: BC817, Package_TO_SOT_SMD:SOT-23, F.Cu at (273.5, 72.9)
- added Q5: BC807, Package_TO_SOT_SMD:SOT-23, F.Cu at (267.7, 84.3)
- added Q6: BC817, Package_TO_SOT_SMD:SOT-23, F.Cu at (263.3, 83.0)
- added Q7: FR9024N, Package_TO_SOT_SMD:TO-252-3_TabPin2, F.Cu at (249.4, 71.4)
- added Q8: FR024N, Package_TO_SOT_SMD:TO-252-3_TabPin2, F.Cu at (249.4, 79.4)
- added R1: 1k, Resistor_SMD:R_1206_3216Metric, F.Cu at (85.9, 34.8)
- added R1: 100k, Resistor_SMD:R_1206_3216Metric, F.Cu at (268.5, 75.8)
- added R2: 1k, Resistor_SMD:R_1206_3216Metric, F.Cu at (85.9, 38.1)
- added R24: 100k, Resistor_SMD:R_1206_3216Metric, F.Cu at (262.9, 75.8)
- added R25: 100k, Resistor_SMD:R_1206_3216Metric, F.Cu at (268.5, 72.5)
- added R26: 4.7k, Resistor_SMD:R_1206_3216Metric, F.Cu at (263.8, 98.8)
- added R27: 33k, Resistor_SMD:R_1206_3216Metric, F.Cu at (258.2, 105.4)
- added R28: 33k, Resistor_SMD:R_1206_3216Metric, F.Cu at (269.0, 95.0)
- added R29: 10k, Resistor_SMD:R_1206_3216Metric, F.Cu at (251.7, 107.8)
- added R3: 10k, Resistor_SMD:R_1206_3216Metric, F.Cu at (91.5, 34.8)
- added R3: 100k, Resistor_SMD:R_1206_3216Metric, F.Cu at (274.6, 69.0)
- added R30: 2.7k, Resistor_SMD:R_1206_3216Metric, F.Cu at (258.2, 102.1)
- added R31: 100k, Resistor_SMD:R_1206_3216Metric, F.Cu at (269.0, 91.7)
- added R32: 33k, Resistor_SMD:R_1206_3216Metric, F.Cu at (258.2, 98.8)
- added R33: 4.7k, Resistor_SMD:R_1206_3216Metric, F.Cu at (246.1, 107.8)
- added R34: 100k, Resistor_SMD:R_1206_3216Metric, F.Cu at (274.6, 91.7)
- added R35: 4.7k, Resistor_SMD:R_1206_3216Metric, F.Cu at (284.2, 85.1)
- added R36: 33k, Resistor_SMD:R_1206_3216Metric, F.Cu at (296.3, 76.1)
- added R37: 33k, Resistor_SMD:R_1206_3216Metric, F.Cu at (307.1, 69.0)
- added R38: 10k, Resistor_SMD:R_1206_3216Metric, F.Cu at (296.3, 79.4)
- added R39: 2.7k, Resistor_SMD:R_1206_3216Metric, F.Cu at (289.8, 85.1)
- added R4: 10k, Resistor_SMD:R_1206_3216Metric, F.Cu at (91.5, 38.1)
- added R4: 33k, Resistor_SMD:R_1206_3216Metric, F.Cu at (256.9, 85.1)
- added R40: 100k, Resistor_SMD:R_1206_3216Metric, F.Cu at (307.1, 72.3)
- added R41: 33k, Resistor_SMD:R_1206_3216Metric, F.Cu at (296.3, 82.7)
- added R42: 4.7k, Resistor_SMD:R_1206_3216Metric, F.Cu at (302.0, 76.1)
- added R43: 100k, Resistor_SMD:R_1206_3216Metric, F.Cu at (312.7, 69.0)
- added R5: 33k, Resistor_SMD:R_1206_3216Metric, F.Cu at (258.2, 79.7)
- added R6: 10k, Resistor_SMD:R_1206_3216Metric, F.Cu at (262.9, 72.5)
- added R8: 4.7k, Resistor_SMD:R_1206_3216Metric, F.Cu at (269.0, 69.0)
- added R9: 4.7k, Resistor_SMD:R_1206_3216Metric, F.Cu at (263.8, 79.1)
